File: Post-Parcial/01-Laboratorio3/Juego/Plano.kicad_pcb (KiCad board)
At the start: 2 copper layers, 32 parts, among them J1 Conn_01x12, J2 Conn_01x12, J3 Conn_01x19, J4 Conn_01x19, Q1 2N3904, Q2 2N3904, Q3 2N3904, Q4 2N3904, Q5 2N3904, Q6 2N3904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

Commit message: Migracion a Kicad8
Parts:
- moved Q4 5.59 mm to (134.1, 92.6)

Commit message: Finalizacion PCB Juego
Parts:
- moved Q7 24.1 mm to (140.7, 126.3)
- moved Q6 23.0 mm to (140.5, 106.1)
- moved Q3 16.0 mm to (136.1, 78.4)
- moved Q9 14.8 mm to (140.6, 112.2)
- moved R14 12.3 mm to (191.1, 106.3)
- moved Q4 6.64 mm to (136.2, 86.3)
- moved Q5 4.84 mm to (140.7, 118.7)
- moved R4 4.36 mm to (159.6, 82.7)
Connections:
- SW1 pad 1: 3.3V -> GND
- SW2 pad 2: 3.3V -> GND
Routing:
- net GND: track 0.00 -> 265.4 mm
- net GPIO13: track 0.00 -> 118.1 mm
- net Net-(Q8-B): track 0.00 -> 95.9 mm
- net GPIO14: track 0.00 -> 95.0 mm
- net GPIO26: track 0.00 -> 79.7 mm
- net Net-(Q3-B): track 0.00 -> 63.4 mm
- net Net-(Q7-B): track 0.00 -> 56.4 mm
- net Net-(Q6-B): track 0.00 -> 53.0 mm
- net GPIO33: track 0.00 -> 44.8 mm
- net GPIO5: track 0.00 -> 40.1 mm
- net Net-(Q9-B): track 0.00 -> 37.6 mm
- net Net-(Q4-B): track 0.00 -> 37.2 mm
- net Net-(Q5-B): track 0.00 -> 36.1 mm
- net GPIO32: track 0.00 -> 34.2 mm
- net Net-(J2-Pin_6): track 0.00 -> 29.0 mm
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