File: Post-Parcial/01-Laboratorio3/Juego/Plano.kicad_sch (KiCad schematic)
At the start: 32 parts, among them J1 Conn_01x12, J2 Conn_01x12, J3 Conn_01x19, J4 Conn_01x19, Q1 2N3904, Q2 2N3904, Q3 2N3904, Q4 2N3904, Q5 2N3904, Q6 2N3904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

Commit message: Finalizacion PCB Juego
Connections:
- net 3.3V: no longer SW1.1, SW2.2
- net GND: now also SW1.1, SW2.2
Other:
- moved on the sheet: SW1
Changed lines of the file:
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@@
 		)
 	)
-	(global_label "3.3V"
-		(shape input)
-		(at 161.29 38.735 180)
-		(fields_autoplaced yes)
-		(effects
-			(font
-				(size 1.27 1.27)
-			)
-			(justify right)
-		)
-		(property "Intersheetrefs" "${INTERSHEET_REFS}"
-			(at 154.1924 38.735 0)
-			(effects
-				(font
-					(size 1.27 1.27)
-				)
-				(justify right)
-				(hide yes)
-			)
-		)
-	)
 	(global_label "GND"
 		(shape input)
@@
 	(global_label "GPIO18"
 		(shape input)
-		(at 171.45 38.735 0)
+		(at 170.942 38.608 0)
 		(fields_autoplaced yes)
 		(effects
@@
 		)
 		(property "Intersheetrefs" "${INTERSHEET_REFS}"
-			(at 181.3295 38.735 0)
+			(at 180.8215 38.608 0)
 			(effects
 				(font
@@
 		)
 	)
+	(global_label "GND"
+		(shape input)
+		(at 163.83 139.7 180)
+		(fields_autoplaced yes)
+		(effects
+			(font
+				(size 1.27 1.27)
+			)
+			(justify right)
+		)
+		(property "Intersheetrefs" "${INTERSHEET_REFS}"
+			(at 156.9743 139.7 0)
+			(effects
+				(font
+					(size 1.27 1.27)
+				)
+				(justify right)
+				(hide yes)
+			)
+		)
+	)
 	(global_label "GPIO23"
 		(shape input)
@@
 		)
 	)
+	(global_label "GND"
+		(shape input)
+		(at 160.782 38.608 180)
+		(fields_autoplaced yes)
+		(effects
+			(font
+				(size 1.27 1.27)
+			)
+			(justify right)
+		)
+		(property "Intersheetrefs" "${INTERSHEET_REFS}"
+			(at 153.9263 38.608 0)
+			(effects
+				(font
+					(size 1.27 1.27)
+				)
+				(justify right)
+				(hide yes)
+			)
+		)
+	)
 	(global_label "GPIO18"
 		(shape input)
@@
 		)
 	)
-	(global_label "3.3V"
-		(shape input)
-		(at 163.83 139.7 180)
-		(fields_autoplaced yes)
-		(effects
-			(font
-				(size 1.27 1.27)
-			)
-			(justify right)
-		)
-		(property "Intersheetrefs" "${INTERSHEET_REFS}"
-			(at 156.7324 139.7 0)
-			(effects
-				(font
-					(size 1.27 1.27)
-				)
-				(justify right)
-				(hide yes)
-			)
-		)
-	)
 	(global_label "GND"
 		(shape input)
@@
 	(symbol
 		(lib_id "Switch:SW_Push")
-		(at 166.37 38.735 0)
+		(at 165.862 38.608 0)
 		(unit 1)
 		(exclude_from_sim no)
@@
 		(fields_autoplaced yes)
 		(property "Reference" "SW1"
-			(at 166.37 31.115 0)
+			(at 165.862 30.988 0)
 			(effects
 				(font
@@
 		)
 		(property "Value" "SW_Push"
-			(at 166.37 33.655 0)
+			(at 165.862 33.528 0)
 			(effects
 				(font
@@
 		)
 		(property "Footprint" "Button_Switch_THT:SW_DIP_SPSTx01_Piano_10.8x4.1mm_W7.62mm_P2.54mm"
-			(at 166.37 33.655 0)
+			(at 165.862 33.528 0)
 			(effects
 				(font
@@
 		)
 		(property "Datasheet" "~"
-			(at 166.37 33.655 0)
+			(at 165.862 33.528 0)
 			(effects
 				(font
@@
 		)
 		(property "Description" ""
-			(at 166.37 38.735 0)
+			(at 165.862 38.608 0)
 			(effects
 				(font
