File: Post-Parcial/Juego - Pruebas/Plano.kicad_pcb (KiCad board)
At the start: 2 copper layers, 33 parts, among them J1 Conn_01x12, J2 Conn_01x12, J3 Conn_01x19, J4 Conn_01x19, Q1 2N3904, Q2 2N3904, Q3 2N3904, Q4 2N3904, Q5 2N3904, Q6 2N3904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

Commit message: Cambios en Prueba PCB Juego
Parts:
- moved Q8 43.2 mm to (148.8, 128.5)
- moved R4 34.7 mm to (191.0, 97.3)
- moved Q2 30.5 mm to (143.8, 78.2)
- moved Q3 18.5 mm to (143.8, 95.2)
- moved Q7 8.98 mm to (148.8, 122.5)
- moved Q5 8.57 mm to (148.8, 116.0)
- moved Q9 8.57 mm to (148.7, 109.5)
- moved Q6 8.57 mm to (148.6, 103.4)
- moved R8 8.38 mm to (173.5, 85.3)
- moved Q4 7.61 mm to (143.8, 87.1)
Routing:
- net GND: track 265.4 -> 0.28 mm
- net GPIO13: track 118.1 -> 0.00 mm
- net Net-(Q8-B): track 95.9 -> 0.00 mm
- net GPIO14: track 95.0 -> 0.00 mm
- net GPIO16: track 90.3 -> 0.00 mm
- net GPIO26: track 79.7 -> 0.00 mm
- net Net-(Q3-B): track 63.4 -> 0.00 mm
- net Net-(Q7-B): track 56.4 -> 0.00 mm
- net Net-(Q6-B): track 53.0 -> 0.00 mm
- net GPIO33: track 44.8 -> 0.00 mm
- net GPIO5: track 40.1 -> 0.00 mm
- net Net-(Q9-B): track 37.6 -> 0.00 mm
- net Net-(Q5-B): track 36.1 -> 0.00 mm
- net Net-(J3-Pin_10): track 34.5 -> 0.00 mm
- net GPIO32: track 34.2 -> 0.00 mm
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
Commit message: Prueba Juego Terminada
Parts:
- R13, R17, R8: footprint Resistor_THT:R_Axial_DIN0204_L3.6mm_D1.6mm_P5.08mm_Horizontal -> Resistor_THT:R_Axial_DIN0309_L9.0mm_D3.2mm_P2.54mm_Vertical
- SW3: footprint Button_Switch_THT:SW_E-Switch_EG1224_SPDT_Angled -> Button_Switch_THT:SW_DIP_SPSTx01_Slide_6.7x4.1mm_W7.62mm_P2.54mm_LowProfile
- moved SW3 92.6 mm to (155.0, 91.8)
- moved Q1 42.2 mm to (148.1, 70.1)
- moved R12 26.5 mm to (188.7, 106.8)
- moved R8 25.8 mm to (198.9, 80.8)
- moved R11 19.4 mm to (193.9, 103.0)
- moved R3 17.0 mm to (193.7, 97.6)
- moved R14 15.5 mm to (191.2, 121.8)
- moved R17 12.9 mm to (178.7, 118.8)
- moved R4 11.9 mm to (191.2, 85.4)
- moved R7 9.89 mm to (192.4, 93.7)
- moved SW1 7.81 mm to (214.5, 76.0)
- moved R13 6.63 mm to (176.1, 103.1)
- moved Q4 5.32 mm to (148.0, 83.9)
- moved Q3 5.11 mm to (148.0, 92.4)
- moved Q2 4.26 mm to (148.0, 77.7)
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Connections:
- J1 pad 7: GPIO16 -> GPIO17
- J3 pad 11: GPIO17 -> Net-(J3-Pin_11)
- J3 pad 12: Net-(J3-Pin_12) -> GPIO16
- Q4 pad 1: GND -> Net-(Q4-E)
- R13 pad 2: Net-(Q5-B) -> Net-(Q6-B)
- R14 pad 2: Net-(Q6-B) -> Net-(Q5-B)
- R3 pad 1: GPIO16 -> GPIO17
- R3 pad 2: Net-(J3-Pin_12) -> Net-(J3-Pin_11)
- R7 pad 1: GPIO17 -> GPIO16
- R8 pad 1: GPIO23 -> unconnected-(R8-Pad1)
- SW3 pad 1: (no net) -> Net-(Q4-E)
- SW3 pad 2: (no net) -> GND
Routing:
- net GND: track 0.28 -> 118.2 mm
- net GPIO13: track 0.00 -> 117.8 mm
- net GPIO14: track 0.00 -> 92.8 mm
- net GPIO26: track 0.00 -> 90.0 mm
- net GPIO17: track 0.00 -> 88.1 mm
- net GPIO5: track 0.00 -> 74.5 mm
- net GPIO33: track 0.00 -> 72.2 mm
- net Net-(Q8-B): track 0.00 -> 53.0 mm
- net Net-(J2-Pin_3): track 0.00 -> 49.4 mm
- net Net-(Q7-B): track 0.00 -> 48.6 mm
- net Net-(Q5-B): track 0.00 -> 44.6 mm
- net Net-(Q1-B): track 101.3 -> 58.8 mm
- net Net-(J1-Pin_3): track 8.74 -> 49.4 mm
- net Net-(J2-Pin_6): track 0.00 -> 37.4 mm
- net Net-(J2-Pin_9): track 0.00 -> 36.1 mm
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