File: Post-Parcial/Juego - Pruebas/Plano.kicad_sch (KiCad schematic)
At the start: 33 parts, among them J1 Conn_01x12, J2 Conn_01x12, J3 Conn_01x19, J4 Conn_01x19, Q1 2N3904, Q2 2N3904, Q3 2N3904, Q4 2N3904, Q5 2N3904, Q6 2N3904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

Commit message: Prueba Juego Terminada
Parts:
- removed SW3: SW_DPST_x2, Button_Switch_THT:SW_E-Switch_EG1224_SPDT_Angled, symbol Switch:SW_DPST_x2
- added SW3: SW_DPST_x2, Button_Switch_THT:SW_DIP_SPSTx01_Slide_6.7x4.1mm_W7.62mm_P2.54mm_LowProfile, symbol Switch:SW_DPST_x2
- R13, R17, R8: footprint Resistor_THT:R_Axial_DIN0204_L3.6mm_D1.6mm_P5.08mm_Horizontal -> Resistor_THT:R_Axial_DIN0309_L9.0mm_D3.2mm_P2.54mm_Vertical
Connections:
- net GND: now also SW3.2 (B); no longer Q4.1 (E)
- net GPIO16: now also J3.12 (Pin_12), R7.1; no longer J1.7 (Pin_7), R3.1
- net GPIO17: now also J1.7 (Pin_7), R3.1; no longer J3.11 (Pin_11), R7.1
- net GPIO23: no longer R8.1
- net at Q6.2 (B): now also R13.2; no longer R14.2
- net at R3.2: now also J3.11 (Pin_11); no longer J3.12 (Pin_12)
- net at Q5.2 (B): now also R14.2; no longer R13.2
- new net: Q4.1 (E), SW3.1 (A)
Other:
- moved on the sheet: J1, Q1, Q2, Q3, Q4, R13, R14, R3, R5, R6, R7, R8
