File: Post-Parcial/Circuitos/CircuitoEjemplos/KiCad8/CircuitoEjemplos.kicad_sch (KiCad schematic)
At the start: 16 parts, among them J1 Conn_01x19, J2 Conn_01x19, SW1 SW_Push, SW2 SW_Push

Commit message: Semestre de Monitoria Finalizado
Connections:
- net GPIO16: no longer R3.1
- net GPIO17: no longer R4.1
- net GPIO18: now also R4.1
- net GPIO5: now also R3.1
Changed lines of the file:
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@@
 		)
 	)
-	(global_label "GPIO16"
+	(global_label "GPIO5"
 		(shape input)
 		(at 166.37 70.358 180)
@@
 		)
 		(property "Intersheetrefs" "${INTERSHEET_REFS}"
-			(at 156.4905 70.358 0)
+			(at 157.7 70.358 0)
 			(effects
 				(font
@@
 		)
 	)
-	(global_label "GPIO17"
+	(global_label "GPIO18"
 		(shape input)
 		(at 166.624 78.486 180)
