File: Post-Parcial/Display 7 segmentos/Plano/Plano.kicad_sch (KiCad schematic)
At the start: 24 parts, among them J3 Conn_01x05, J3 Conn_01x19, J4 Conn_01x05, J4 Conn_01x19, J5 Conn_01x05, J6 Conn_01x05, Q1 2N3904, Q2 2N3904

Commit message: Semestre de Monitoria Finalizado
Parts:
- removed R1, R15, R2, R3, R4, R5, R6: 330, Resistor_THT:R_Axial_DIN0207_L6.3mm_D2.5mm_P2.54mm_Vertical, symbol Device:R
- added R? (x7): 330, Resistor_THT:R_Axial_DIN0207_L6.3mm_D2.5mm_P2.54mm_Vertical, symbol Device:R
- renumbered J3 to J?, J4 to J?
Connections:
- net 5V: no longer Q1.3 (C), Q2.3 (C)
- net GPIO1: no longer J5.4 (Pin_4)
- net GPIO12: no longer J4.4 (Pin_4)
- net GPIO14: no longer J4.2 (Pin_2)
- net GPIO18: now also R?.1; no longer J6.4 (Pin_4), R14.2
- net GPIO19: now also R14.1; no longer J6.2 (Pin_2), R13.2
- net GPIO21: now also R13.1; no longer J6.1 (Pin_1), R12.2
- net GPIO22: no longer J5.2 (Pin_2)
- net GPIO23: no longer J5.1 (Pin_1)
- net GPIO25: no longer J3.4 (Pin_4)
- net GPIO26: no longer J3.5 (Pin_5)
- net GPIO27: no longer J4.1 (Pin_1)
- net GPIO3: no longer J5.5 (Pin_5)
- net GPIO32: no longer J3.1 (Pin_1)
- net GPIO33: no longer J3.2 (Pin_2)
- net at R7.1: now also J5.1 (Pin_1)
- net at R11.1: now also J5.5 (Pin_5)
- net at J6.3 (Pin_3): no longer Q2.1 (E)
- net at J6.5 (Pin_5): now also R?.2
- net at J4.3 (Pin_3): no longer Q1.1 (E)
- net at R10.1: now also J5.4 (Pin_4)
- net at R9.1: now also J5.2 (Pin_2)
- new net: J6.2 (Pin_2), R14.2
- new net: J4.1 (Pin_1), R?.2
- new net: J6.1 (Pin_1), R13.2
- new net: J6.4 (Pin_4), R?.2
- new net: J4.2 (Pin_2), R?.2
- no-connect marks 11 -> 10
Other:
- moved on the sheet: J3, J4, J5, J6, Q1, Q2, R16, R8
